Commit message: dual arm launcher

File: iiwa_description/gazebo/iiwa.gazebo.xacro (robot description, xacro)
@@ -14,8 +14,4 @@
       </plugin>
     </gazebo>
-    <!-- color -->
-    <gazebo reference="${prefix}link_7">
-      <material>Gazebo/Gray</material>
-    </gazebo>
   </xacro:macro>
 </robot>
