Commit message: srdf

File: iiwa_description/srdf/iiwa_dual.srdf.xacro (robot description, xacro)
@@ -10,4 +10,13 @@
   <disable_collisions link1="marker_link_0" link2="r_link_7" reason="Adjacent" />
   <disable_collisions link1="marker_link_0" link2="r_link_6" reason="Adjacent" />
+  <group_state name="calibration" group="r_iiwa_arm">
+        <joint name="r_joint_a1" value="-0.8002797903942479"/>
+        <joint name="r_joint_a2" value="-0.9500586171190173"/>
+        <joint name="r_joint_a3" value="0.1643627515424193"/>
+        <joint name="r_joint_a4" value="1.7912287728082115"/>
+        <joint name="r_joint_a5" value="-0.7668156360694677"/>
+        <joint name="r_joint_a6" value="1.1804337818299833"/>
+        <joint name="r_joint_a7" value="0.17710744409784557"/>
+ </group_state>
   <xacro:iiwa_srdf name="$(arg name)" prefix="l_" base="base"/>
   <xacro:iiwa_srdf name="$(arg name)" prefix="r_" base="base"/>
