Commit message: config

File: iiwa_description/srdf/iiwa_dual_macro.srdf.xacro (robot description, xacro)
@@ -13,4 +13,13 @@
         <joint name="${prefix}joint_a6" value="1.571"/>
         <joint name="${prefix}joint_a7" value="0.785"/>
+    </group_state>
+     <group_state name="upright" group="${prefix}${name}_arm">
+        <joint name="${prefix}joint_a1" value="0"/>
+        <joint name="${prefix}joint_a2" value="0"/>
+        <joint name="${prefix}joint_a3" value="0"/>
+        <joint name="${prefix}joint_a4" value="0"/>
+        <joint name="${prefix}joint_a5" value="0"/>
+        <joint name="${prefix}joint_a6" value="0"/>
+        <joint name="${prefix}joint_a7" value="0"/>
     </group_state>
     <disable_collisions link1="${base}" link2="${prefix}link_0" reason="Adjacent" />
