Commit message: gripper plate

File: iiwa_description/config/iiwa.config.xacro (robot description, xacro)
@@ -18,4 +18,10 @@
     <!-- Import iiwa urdf file -->
     <xacro:include filename="$(find ${description_package})/urdf/iiwa.urdf.xacro" />
+    <xacro:if value="${show_aruco_board}">
+    	<xacro:generic_aruco aruco_dictionary="DICT_4X4_50" aruco_id="1" aruco_l="0.2" aruco_name="marker" white_border="${50 * 0.2/700}" connected_to="r_tool0">
+        <!-- fake origin not needed! when origin is not specified!-->
+       	 <origin xyz="0 0.0 0.1" rpy="0 1.57 0" />
+    	</xacro:generic_aruco>
+   </xacro:if>
     <!-- Import iiwa ros2_control description -->
     <xacro:include filename="$(find ${description_package})/ros2_control/iiwa.r2c_hardware.xacro" />

File: iiwa_description/config/iiwa_dual.config.xacro (robot description, xacro)
@@ -15,7 +15,9 @@
     <xacro:arg name="controllers_file" default="iiwa_dual_controllers.yaml" />
     <xacro:arg name="show_aruco_board" default="false" />
+    <xacro:arg name="add_gripper_links" default="true" />
     <xacro:arg name="namespace" default="/" />
     <xacro:property name="description_package" value="$(arg description_package)"/>
     <xacro:property name="show_aruco_board" value="$(arg show_aruco_board)"/>
+    <xacro:property name="add_gripper_links" value="$(arg add_gripper_links)"/>
     <!-- Import iiwa urdf file -->
     <xacro:include filename="$(find ${description_package})/urdf/iiwa_dual.urdf.xacro" />
@@ -140,9 +142,9 @@
        <origin xyz="-0.025 0 0" rpy="-1.57 0 1.57" />
     </joint>
-    <xacro:iiwa parent="base" prefix="l_">
+    <xacro:iiwa parent="base" prefix="l_" add_gripper_link="${add_gripper_links}">
         <origin xyz="${left_base_frame['x']} ${left_base_frame['y']} ${left_base_frame['z']}"
             rpy="${left_base_frame['roll']} ${left_base_frame['pitch']} ${left_base_frame['yaw']}" />
     </xacro:iiwa>
-    <xacro:iiwa parent="base" prefix="r_">
+    <xacro:iiwa parent="base" prefix="r_" add_gripper_link="${add_gripper_links}">
         <origin xyz="${right_base_frame['x']} ${right_base_frame['y']} ${right_base_frame['z']}"
             rpy="${right_base_frame['roll']} ${right_base_frame['pitch']} ${right_base_frame['yaw']}" />

File: iiwa_description/srdf/iiwa_dual_macro.srdf.xacro (robot description, xacro)
@@ -47,4 +47,5 @@
     <disable_collisions link1="${prefix}link_6" link2="${prefix}link_7" reason="Adjacent" />
     <disable_collisions link1="${prefix}link_7" link2="${prefix}tool0" reason="Adjacent" />
+    <disable_collisions link1="${prefix}tool0" link2="${prefix}gripper" reason="Adjacent" />
   </xacro:macro>
 </robot>

File: iiwa_description/urdf/iiwa_dual.urdf.xacro (robot description, xacro)
@@ -1,5 +1,8 @@
 <?xml version="1.0"?>
 <robot xmlns:xacro="http://www.ros.org/wiki/xacro">
-  <xacro:macro name="iiwa" params="parent prefix *origin">
+  <xacro:macro name="iiwa" params="parent prefix add_gripper_link *origin">
+<xacro:property name="gripper_length" value="0.15" />
+<xacro:property name="gripper_width" value="0.1" />
+<xacro:property name="gripper_depth" value="0.01" />
   <link name="${prefix}iiwa_base" type="fixed"/>
   <joint name="${prefix}iiwa_root_joint" type="fixed">
@@ -222,4 +225,41 @@
       <axis xyz="0 0 0"/>
   </joint>
+   <xacro:if value="${add_gripper_link}">
+        <link name="${prefix}gripper">
+            <visual>
+                <origin xyz="0 0 ${gripper_length/2}" rpy="0 0 0" />
+                <geometry>
+                    <box size="${gripper_width} ${gripper_depth} ${gripper_length}" />
+                </geometry>
+                <material name="White">
+                    <color rgba="1.0 1.0 1.0 1.0" />
+                </material>
+            </visual>
+            <collision>
+                 <origin xyz="0 0 ${gripper_length/2}" rpy="0 0 0" />
+                <geometry>
+                    <box size="${gripper_width} ${gripper_depth} ${gripper_length}" />
+                </geometry>
+            </collision>
+            <inertial>
+            <origin xyz="0.0 0.0 0.0" rpy="0.0 0.0 0.0"/>
+            <mass value="10.0"/>
+            <inertia ixx="0.001" ixy="0.0" ixz="0.001" iyy="0.0" iyz="0.0" izz="0.001"/>
+            </inertial>
+    	 </link>
+        <joint name="${prefix}joint_tool0_gripper" type="fixed">
+            <origin rpy="0 0 0" xyz="0 0 0"/>
+            <parent link="${prefix}tool0"/>
+             <child link="${prefix}gripper"/>
+             <axis xyz="0 0 0"/>
+         </joint>
+         <link name="${prefix}ee"/>
+          <joint name="${prefix}joint_gripper_ee" type="fixed">
+            <origin xyz="0 0 ${gripper_length}" rpy="0 0 0"/>
+            <parent link="${prefix}gripper"/>
+             <child link="${prefix}ee"/>
+             <axis xyz="0 0 0"/>
+         </joint>
+   </xacro:if>
   </xacro:macro>
 </robot>
