Commit message: camera axis

File: iiwa_description/config/iiwa_dual.config.xacro (robot description, xacro)
@@ -105,16 +105,14 @@
     <link name="camera">
         <visual>
-            <origin xyz="-0.025 0 1.15" rpy="0 -0.8 0" />
             <geometry>
-                <box size="0.05 0.1 0.05" />
+                <box size="0.02 0.1 0.05" />
             </geometry>
             <material name="Red">
-                <color rgba="1.0 0.0 0.0 1.0" />
+                <color rgba="0.5 0.0 0.5 1.0" />
             </material>
         </visual>
         <collision>
-            <origin xyz="0 0 0.6" rpy="0 0 0" />
-            <geometry>
-                <box size="0.025 0.025 1.2" />
+             <geometry>
+                <box size="0.02 0.1 0.05" />
             </geometry>
         </collision>
@@ -128,5 +126,11 @@
         <parent link="camera_pole"/>
         <child link="camera"/>
-        <origin xyz="0.0 0.0 0.0" rpy="0.0 0.0 0.0"/>
+       <origin xyz="-0.025 0 1.15" rpy="0 -0.8 0" />
+    </joint>
+    <link name="camera_optical_frame"/>
+     <joint name="camera_optical_frame_to_camera" type="fixed">
+        <parent link="camera"/>
+        <child link="camera_optical_frame"/>
+       <origin xyz="-0.025 0 0" rpy="1.57 0 -1.57" />
     </joint>
     <xacro:iiwa parent="base" prefix="l_">

Commit message: aruco

File: iiwa_description/config/iiwa_dual.config.xacro (robot description, xacro)
@@ -44,5 +44,5 @@
     <color rgba="0.5 0.5 0.5 1.0"/>
     </material>
-    <xacro:generic_aruco aruco_dictionary="DICT_4X4_50" aruco_id="1" aruco_l="0.1" aruco_name="marker" white_border="0.01" connected_to="r_link_7">
+    <xacro:generic_aruco aruco_dictionary="DICT_4X4_50" aruco_id="1" aruco_l="0.1" aruco_name="marker" white_border="0.1" connected_to="r_link_7">
         <!-- fake origin not needed! when origin is not specified!-->
         <origin xyz="0.06 0.0 0.1" rpy="0 1.57 0" />
@@ -132,5 +132,5 @@
         <parent link="camera"/>
         <child link="camera_optical_frame"/>
-       <origin xyz="-0.025 0 0" rpy="1.57 0 -1.57" />
+       <origin xyz="-0.025 0 0" rpy="-1.57 0 1.57" />
     </joint>
     <xacro:iiwa parent="base" prefix="l_">

File: iiwa_description/urdf/aruco.urdf.xacro (robot description, xacro)
@@ -32,4 +32,7 @@
           <box size="${aruco_l + 2*white_border * aruco_l} ${aruco_l + 2*white_border * aruco_l} ${0.01 * aruco_l/0.09}"/>
         </geometry>
+         <material name="white">
+	    <color rgba="1 1 1 1"/>
+	  </material>
       </visual>
       <visual>

Commit message: aruco marker

File: iiwa_description/config/iiwa_dual.config.xacro (robot description, xacro)
@@ -46,5 +46,5 @@
     <xacro:generic_aruco aruco_dictionary="DICT_4X4_50" aruco_id="1" aruco_l="0.1" aruco_name="marker" white_border="0.1" connected_to="r_link_7">
         <!-- fake origin not needed! when origin is not specified!-->
-        <origin xyz="0.06 0.0 0.1" rpy="0 1.57 0" />
+        <origin xyz="0.06 0.0 0.15" rpy="0 1.57 0" />
     </xacro:generic_aruco>
  <!-- table as base for the 2 iiwa's -->

Commit message: aruco

File: iiwa_description/config/iiwa_dual.config.xacro (robot description, xacro)
@@ -44,5 +44,5 @@
     <color rgba="0.5 0.5 0.5 1.0"/>
     </material>
-    <xacro:generic_aruco aruco_dictionary="DICT_4X4_50" aruco_id="1" aruco_l="0.1" aruco_name="marker" white_border="0.1" connected_to="r_link_7">
+    <xacro:generic_aruco aruco_dictionary="DICT_4X4_50" aruco_id="1" aruco_l="0.2" aruco_name="marker" white_border="0.01" connected_to="r_link_7">
         <!-- fake origin not needed! when origin is not specified!-->
         <origin xyz="0.06 0.0 0.15" rpy="0 1.57 0" />

File: iiwa_description/urdf/aruco.urdf.xacro (robot description, xacro)
@@ -40,5 +40,5 @@
         <geometry>
           <!-- <box size="0.09 0.09 0.01"/> -->
-          <mesh filename="package://iiwa_description/meshes/aruco/${aruco_dictionary}/${aruco_dictionary}_id${aruco_id}.dae" scale="${aruco_l/0.09} ${aruco_l/0.09} ${aruco_l/0.09}"/>
+          <mesh filename="package://iiwa_description/meshes/aruco/aruco.dae" scale="${aruco_l/0.09} ${aruco_l/0.09} ${aruco_l/0.09}"/>
         </geometry>
       </visual>

Commit message: calibration target

File: iiwa_description/config/iiwa_dual.config.xacro (robot description, xacro)
@@ -44,7 +44,7 @@
     <color rgba="0.5 0.5 0.5 1.0"/>
     </material>
-    <xacro:generic_aruco aruco_dictionary="DICT_4X4_50" aruco_id="1" aruco_l="0.2" aruco_name="marker" white_border="0.01" connected_to="r_link_7">
+    <xacro:generic_aruco aruco_dictionary="DICT_4X4_50" aruco_id="1" aruco_l="0.2" aruco_name="marker" white_border="${50 * 0.2/700}" connected_to="r_tool0">
         <!-- fake origin not needed! when origin is not specified!-->
-        <origin xyz="0.06 0.0 0.15" rpy="0 1.57 0" />
+        <origin xyz="0 0.0 0.1" rpy="0 1.57 0" />
     </xacro:generic_aruco>
  <!-- table as base for the 2 iiwa's -->

File: iiwa_description/srdf/iiwa_dual.srdf.xacro (robot description, xacro)
@@ -11,11 +11,11 @@
   <disable_collisions link1="marker_link_0" link2="r_link_6" reason="Adjacent" />
   <group_state name="calibration" group="r_iiwa_arm">
-        <joint name="r_joint_a1" value="-0.8002797903942479"/>
-        <joint name="r_joint_a2" value="-0.9500586171190173"/>
-        <joint name="r_joint_a3" value="0.1643627515424193"/>
-        <joint name="r_joint_a4" value="1.7912287728082115"/>
-        <joint name="r_joint_a5" value="-0.7668156360694677"/>
-        <joint name="r_joint_a6" value="1.1804337818299833"/>
-        <joint name="r_joint_a7" value="0.17710744409784557"/>
+        <joint name="r_joint_a1" value="-0.08010961654547082"/>
+        <joint name="r_joint_a2" value="-0.16420504552657098"/>
+        <joint name="r_joint_a3" value="-0.27250731500631165"/>
+        <joint name="r_joint_a4" value="1.8724710663682194"/>
+        <joint name="r_joint_a5" value="1.2174080270970293"/>
+        <joint name="r_joint_a6" value="1.2045682076607263"/>
+        <joint name="r_joint_a7" value="-0.11062877843161172"/>
  </group_state>
   <xacro:iiwa_srdf name="$(arg name)" prefix="l_" base="base"/>

File: iiwa_description/urdf/aruco.urdf.xacro (robot description, xacro)
@@ -24,5 +24,5 @@
         <origin xyz="0 0 0" rpy="0 0 0"/>
         <geometry>
-          <box size="${aruco_l + 2*white_border * aruco_l} ${aruco_l + 2*white_border * aruco_l} ${0.01 * aruco_l/0.09}"/>
+          <box size="${aruco_l} ${aruco_l} ${0.01 * aruco_l/0.09}"/>
         </geometry>
       </collision>
@@ -30,5 +30,5 @@
         <origin xyz="0 0 0" rpy="0 0 0"/>
         <geometry>
-          <box size="${aruco_l + 2*white_border * aruco_l} ${aruco_l + 2*white_border * aruco_l} ${0.01 * aruco_l/0.09}"/>
+          <box size="${aruco_l} ${aruco_l} ${0.01 * aruco_l/0.09}"/>
         </geometry>
          <material name="white">
@@ -44,4 +44,10 @@
       </visual>
     </link>
+    <link name="${aruco_name}_link_origin" />
+    <joint name="${aruco_name}_joint_origin_link0" type="fixed">
+    <parent link = "${aruco_name}_link_0"/>
+    <child link= "${aruco_name}_link_origin" />
+    <origin xyz="${aruco_l/2 - white_border} ${aruco_l/2 - white_border} ${0.005 * aruco_l/0.09}" rpy="0 0 3.14"/>
+    </joint>
     <gazebo reference="${aruco_name}_link_0">
       <kp>100000.0</kp>

Commit message: aruco board switch

File: iiwa_description/config/iiwa_dual.config.xacro (robot description, xacro)
@@ -14,6 +14,8 @@
     <xacro:arg name="runtime_config_package" default="iiwa_description" />
     <xacro:arg name="controllers_file" default="iiwa_dual_controllers.yaml" />
+    <xacro:arg name="show_aruco_board" default="false" />
     <xacro:arg name="namespace" default="/" />
     <xacro:property name="description_package" value="$(arg description_package)"/>
+    <xacro:property name="show_aruco_board" value="$(arg show_aruco_board)"/>
     <!-- Import iiwa urdf file -->
     <xacro:include filename="$(find ${description_package})/urdf/iiwa_dual.urdf.xacro" />
@@ -22,5 +24,7 @@
     <!-- Import all Gazebo-customization elements -->
     <xacro:include filename="$(find ${description_package})/gazebo/iiwa.gazebo.xacro"/>
-    <xacro:include filename="$(find ${description_package})/urdf/aruco.urdf.xacro"/>
+    <xacro:if value="${show_aruco_board}">
+    	<xacro:include filename="$(find ${description_package})/urdf/aruco.urdf.xacro"/>
+    </xacro:if>
     <!-- Used for fixing robot -->
     <link name="world"/>
@@ -44,8 +48,10 @@
     <color rgba="0.5 0.5 0.5 1.0"/>
     </material>
-    <xacro:generic_aruco aruco_dictionary="DICT_4X4_50" aruco_id="1" aruco_l="0.2" aruco_name="marker" white_border="${50 * 0.2/700}" connected_to="r_tool0">
+    <xacro:if value="${show_aruco_board}">
+    	<xacro:generic_aruco aruco_dictionary="DICT_4X4_50" aruco_id="1" aruco_l="0.2" aruco_name="marker" white_border="${50 * 0.2/700}" connected_to="r_tool0">
         <!-- fake origin not needed! when origin is not specified!-->
-        <origin xyz="0 0.0 0.1" rpy="0 1.57 0" />
-    </xacro:generic_aruco>
+       	 <origin xyz="0 0.0 0.1" rpy="0 1.57 0" />
+    	</xacro:generic_aruco>
+   </xacro:if>
  <!-- table as base for the 2 iiwa's -->
     <link name="base">

File: iiwa_description/srdf/iiwa_dual.srdf.xacro (robot description, xacro)
@@ -4,8 +4,11 @@
   <xacro:arg name="prefix" default="" />
   <xacro:arg name="description_package" default="iiwa_description" />
+  <xacro:arg name="show_aruco_board" default="false" />
   <xacro:property name="description_package" value="$(arg description_package)"/>
+   <xacro:property name="show_aruco_board" value="$(arg show_aruco_board)"/>
   <xacro:include filename="$(find ${description_package})/srdf/iiwa_dual_macro.srdf.xacro"/>
   <disable_collisions link1="base" link2="camera_pole" reason="Adjacent" />
   <disable_collisions link1="camera" link2="camera_pole" reason="Adjacent" />
+  <xacro:if value="${show_aruco_board}">
   <disable_collisions link1="marker_link_0" link2="r_link_7" reason="Adjacent" />
   <disable_collisions link1="marker_link_0" link2="r_link_6" reason="Adjacent" />
@@ -19,4 +22,5 @@
         <joint name="r_joint_a7" value="-0.11062877843161172"/>
  </group_state>
+  </xacro:if>
   <xacro:iiwa_srdf name="$(arg name)" prefix="l_" base="base"/>
   <xacro:iiwa_srdf name="$(arg name)" prefix="r_" base="base"/>

Commit message: realsense camera

File: iiwa_description/config/iiwa_dual.config.xacro (robot description, xacro)
@@ -29,4 +29,5 @@
     	<xacro:include filename="$(find ${description_package})/urdf/aruco.urdf.xacro"/>
     </xacro:if>
+    <xacro:include filename="$(find ${description_package})/urdf/d435.urdf.xacro"/>
     <!-- Used for fixing robot -->
     <link name="world"/>
@@ -111,4 +112,7 @@
         <origin xyz="0.0 0.0 0.0" rpy="0.0 0.0 0.0"/>
     </joint>
+    <xacro:sensor_d435 parent="camera_pole" >
+        <origin xyz="-0.025 0 1.15" rpy="0 0.8 3.14"/>
+    </xacro:sensor_d435>
     <link name="camera">
         <visual>

Commit message: realsense camera

File: iiwa_description/config/iiwa_dual.config.xacro (robot description, xacro)
@@ -113,6 +113,7 @@
     </joint>
     <xacro:sensor_d435 parent="camera_pole" >
-        <origin xyz="-0.025 0 1.15" rpy="0 0.8 3.14"/>
+        <origin xyz="-0.025 0.01 1.15" rpy="0 0.8 3.14"/>
     </xacro:sensor_d435>
+<!--
     <link name="camera">
         <visual>
@@ -146,4 +147,5 @@
        <origin xyz="-0.025 0 0" rpy="-1.57 0 1.57" />
     </joint>
+-->
     <xacro:iiwa parent="base" prefix="l_" add_gripper_link="${add_gripper_links}">
         <origin xyz="${left_base_frame['x']} ${left_base_frame['y']} ${left_base_frame['z']}"

File: iiwa_description/srdf/iiwa_dual.srdf.xacro (robot description, xacro)
@@ -9,5 +9,5 @@
   <xacro:include filename="$(find ${description_package})/srdf/iiwa_dual_macro.srdf.xacro"/>
   <disable_collisions link1="base" link2="camera_pole" reason="Adjacent" />
-  <disable_collisions link1="camera" link2="camera_pole" reason="Adjacent" />
+  <disable_collisions link1="camera_link" link2="camera_pole" reason="Adjacent" />
   <xacro:if value="${show_aruco_board}">
   <disable_collisions link1="marker_link_0" link2="r_link_7" reason="Adjacent" />
@@ -26,6 +26,6 @@
   <xacro:iiwa_srdf name="$(arg name)" prefix="r_" base="base"/>
   <group name="dual_arm">
-    <group name="l_iiwa_arm_ee" />
-    <group name="r_iiwa_arm_ee" />
+    <group name="l_iiwa_arm" />
+    <group name="r_iiwa_arm" />
   </group>
 </robot>

Commit message: camera fix

File: iiwa_description/config/iiwa_dual.config.xacro (robot description, xacro)
@@ -112,9 +112,10 @@
         <origin xyz="0.0 0.0 0.0" rpy="0.0 0.0 0.0"/>
     </joint>
+    <!--
     <xacro:sensor_d435 parent="camera_pole" >
         <origin xyz="-0.025 0.01 1.15" rpy="0 0.8 3.14"/>
     </xacro:sensor_d435>
-<!--
-    <link name="camera">
+-->
+    <link name="camera_link">
         <visual>
             <geometry>
@@ -138,14 +139,13 @@
     <joint name="camera_to_pole" type="fixed">
         <parent link="camera_pole"/>
-        <child link="camera"/>
+        <child link="camera_link"/>
        <origin xyz="-0.025 0 1.15" rpy="0 -0.8 0" />
     </joint>
-    <link name="camera_optical_frame"/>
+    <link name="camera_color_optical_frame"/>
      <joint name="camera_optical_frame_to_camera" type="fixed">
-        <parent link="camera"/>
-        <child link="camera_optical_frame"/>
+        <parent link="camera_link"/>
+        <child link="camera_color_optical_frame"/>
        <origin xyz="-0.025 0 0" rpy="-1.57 0 1.57" />
     </joint>
--->
     <xacro:iiwa parent="base" prefix="l_" add_gripper_link="${add_gripper_links}">
         <origin xyz="${left_base_frame['x']} ${left_base_frame['y']} ${left_base_frame['z']}"

Commit message: uc2

File: iiwa_description/config/iiwa_dual.config.xacro (robot description, xacro)
@@ -156,4 +156,30 @@
             rpy="${right_base_frame['roll']} ${right_base_frame['pitch']} ${right_base_frame['yaw']}" />
     </xacro:iiwa>
+        <joint name="l_joint_tool1_plate" type="fixed">
+            <origin rpy="0 0 -1.5708" xyz="0 0 0"/>
+            <parent link="l_tool1"/>
+             <child link="l_plate_link"/>
+             <axis xyz="0 0 0"/>
+         </joint>
+         <link name="l_ee"/>
+          <joint name="l_joint_gripper_ee" type="fixed">
+            <origin xyz="0.027 0 0.168" rpy="0 0.0698 0"/>
+            <parent link="l_plate_link"/>
+             <child link="l_ee"/>
+             <axis xyz="0 0 0"/>
+         </joint>
+           <joint name="r_joint_tool1_plate" type="fixed">
+            <origin rpy="0 0 1.5708" xyz="0 0 0"/>
+            <parent link="r_tool1"/>
+             <child link="r_plate_link"/>
+             <axis xyz="0 0 0"/>
+         </joint>
+         <link name="r_ee"/>
+          <joint name="r_joint_gripper_ee" type="fixed">
+            <origin xyz="0.027 0 0.168" rpy="0 0.0698 0"/>
+            <parent link="r_plate_link"/>
+             <child link="r_ee"/>
+             <axis xyz="0 0 0"/>
+         </joint>
     <xacro:iiwa_r2c_hardware
         name="iiwa_left" prefix="l_"

File: iiwa_description/urdf/iiwa_dual.urdf.xacro (robot description, xacro)
@@ -169,5 +169,52 @@
       </inertial>
   </link>
+   <link name="${prefix}ft_sensor_link">
+    <visual>
+      <origin rpy="3.14159 0.0 0.0" xyz="-0.037 0.037 0.017"/>
+        <geometry>
+        <mesh filename="package://iiwa_description/meshes/ati/ati_gamma.stl" scale="1.0 1.0 1.0"/>
+        </geometry>
+       <material name="Grey">
+                    <color rgba="0.5 0.5 0.5 1.0" />
+                </material>
+    </visual>
+    <!--
+    <collision>
+      <origin rpy="0 0 0" xyz="0.0 0.0 0.017"/>
+      <geometry>
+        <mesh filename="package://iiwa_description/meshes/ati/ati_gamma.stl" scale="1.0 1.0 1.0"/>
+      </geometry>
+    </collision>
+    -->
+    <inertial>
+      <mass value="0.1"/>
+      <origin rpy="0 0 0" xyz="0 0 0.017"/>
+      <inertia ixx="1e-3" ixy="0.0" ixz="0.0" iyy="1e-3" iyz="0.0" izz="1e-3"/>
+    </inertial>
+  </link>
+  <link name="${prefix}plate_link">
+	  <collision>
+		  <geometry>
+		    <mesh filename="package://iiwa_description/meshes/plates/gamma_plate_gripper.stl" scale="0.001 0.001 0.001"/>
+		  </geometry>
+		  <origin rpy="0 0 0.0" xyz="-0.035 -0.05 0.0"/>
+	</collision>
+	<visual>
+		<geometry>
+			<mesh filename="package://iiwa_description/meshes/plates/gamma_plate_gripper.stl" scale="0.001 0.001 0.001"/>
+		</geometry>
+		  <origin rpy="0 0 0" xyz="-0.035 -0.05 0.0"/>
+		  <material name="lc_soft_enable_wide_grip_Base_SWA.stl">
+			  <color rgba="0.4891 0.5125 0.5281 1.0"/>
+		  </material>
+	</visual>
+  <inertial>
+          <inertia ixx="0.0024968641" ixy="0.0" ixz="0.0" iyy="0.0022605853" iyz="0.0" izz="0.0011041847"/>
+          <origin rpy="0 0 0" xyz="0.0 0.0 0.02"/>
+          <mass value="0.6"/>
+  </inertial>
+  </link>
   <link name="${prefix}tool0"/>
+  <link name="${prefix}tool1"/>
   <joint name="${prefix}joint_a1" type="revolute">
       <origin rpy="0 0 0" xyz="0 0 0"/>
@@ -220,46 +267,21 @@
   </joint>
   <joint name="${prefix}joint_a7-tool0" type="fixed">
-      <origin rpy="0 0 0" xyz="0 0 0.154"/>
+      <origin rpy="0 0 0" xyz="0 0 0.152"/>
       <parent link="${prefix}link_7"/>
       <child link="${prefix}tool0"/>
       <axis xyz="0 0 0"/>
   </joint>
-   <xacro:if value="${add_gripper_link}">
-        <link name="${prefix}gripper">
-            <visual>
-                <origin xyz="0 0 ${gripper_length/2}" rpy="0 0 0" />
-                <geometry>
-                    <box size="${gripper_width} ${gripper_depth} ${gripper_length}" />
-                </geometry>
-                <material name="White">
-                    <color rgba="1.0 1.0 1.0 1.0" />
-                </material>
-            </visual>
-            <collision>
-                 <origin xyz="0 0 ${gripper_length/2}" rpy="0 0 0" />
-                <geometry>
-                    <box size="${gripper_width} ${gripper_depth} ${gripper_length}" />
-                </geometry>
-            </collision>
-            <inertial>
-            <origin xyz="0.0 0.0 0.0" rpy="0.0 0.0 0.0"/>
-            <mass value="10.0"/>
-            <inertia ixx="0.001" ixy="0.0" ixz="0.001" iyy="0.0" iyz="0.0" izz="0.001"/>
-            </inertial>
-    	 </link>
-        <joint name="${prefix}joint_tool0_gripper" type="fixed">
-            <origin rpy="0 0 0" xyz="0 0 0"/>
-            <parent link="${prefix}tool0"/>
-             <child link="${prefix}gripper"/>
-             <axis xyz="0 0 0"/>
-         </joint>
-         <link name="${prefix}ee"/>
-          <joint name="${prefix}joint_gripper_ee" type="fixed">
-            <origin xyz="0 0 ${gripper_length}" rpy="0 0 0"/>
-            <parent link="${prefix}gripper"/>
-             <child link="${prefix}ee"/>
-             <axis xyz="0 0 0"/>
-         </joint>
-   </xacro:if>
+  <joint name="${prefix}ft_joint" type="fixed">
+    <origin rpy="0.0 0.0 0" xyz="0.00 0.0 ${0.017}"/>
+    <axis xyz="0 0 1"/>
+    <parent link="${prefix}tool0"/>
+    <child link="${prefix}ft_sensor_link"/>
+  </joint>
+  <joint name="${prefix}ft_joint-tool1" type="fixed">
+    <origin rpy="0.0 0.0 0" xyz="0.00 0.0 ${0.017}"/>
+    <axis xyz="0 0 1"/>
+    <parent link="${prefix}ft_sensor_link"/>
+    <child link="${prefix}tool1"/>
+  </joint>
   </xacro:macro>
 </robot>

Commit message: fixed gripper axes

File: iiwa_description/config/iiwa_dual.config.xacro (robot description, xacro)
@@ -164,5 +164,5 @@
          <link name="l_ee"/>
           <joint name="l_joint_gripper_ee" type="fixed">
-            <origin xyz="0.027 0 0.168" rpy="0 0.0698 0"/>
+            <origin xyz="0.027 0 0.168" rpy="0 0.0698 -1.5708"/>
             <parent link="l_plate_link"/>
              <child link="l_ee"/>
@@ -177,5 +177,5 @@
          <link name="r_ee"/>
           <joint name="r_joint_gripper_ee" type="fixed">
-            <origin xyz="0.027 0 0.168" rpy="0 0.0698 0"/>
+            <origin xyz="0.027 0 0.168" rpy="0 0.0698 1.5708"/>
             <parent link="r_plate_link"/>
              <child link="r_ee"/>

File: iiwa_description/srdf/iiwa_dual_macro.srdf.xacro (robot description, xacro)
@@ -59,5 +59,6 @@
     <disable_collisions link1="${prefix}link_6" link2="${prefix}link_7" reason="Adjacent" />
     <disable_collisions link1="${prefix}link_7" link2="${prefix}tool0" reason="Adjacent" />
-    <disable_collisions link1="${prefix}tool0" link2="${prefix}gripper" reason="Adjacent" />
+    <disable_collisions link1="${prefix}ft_sensor_link" link2="${prefix}link_7" reason="Adjacent" />
+    <disable_collisions link1="${prefix}ft_sensor_link" link2="${prefix}plate_link" reason="Adjacent" />
   </xacro:macro>
 </robot>

File: iiwa_description/urdf/iiwa_dual.urdf.xacro (robot description, xacro)
@@ -179,4 +179,10 @@
                 </material>
     </visual>
+     <collision>
+      <origin rpy="3.14159 0.0 0.0" xyz="-0.037 0.037 0.017"/>
+        <geometry>
+        <mesh filename="package://iiwa_description/meshes/ati/ati_gamma.stl" scale="1.0 1.0 1.0"/>
+        </geometry>
+    </collision>
     <!--
     <collision>
