Commit message: uc2 setup

File: iiwa_description/config/iiwa_dual.config.xacro (robot description, xacro)
@@ -8,5 +8,4 @@
     <xacro:arg name="robot_ip" default="192.170.10.2" />
     <xacro:arg name="robot_port" default="30200" />
-    <xacro:arg name="initial_positions_file" default="initial_positions.yaml" />
     <xacro:arg name="command_interface" default="position" />
     <xacro:arg name="base_frame_file" default="base_frame.yaml" />
@@ -16,8 +15,10 @@
     <xacro:arg name="show_aruco_board" default="false" />
     <xacro:arg name="add_gripper_links" default="true" />
+    <xacro:arg name="add_virtual_camera" default="false" />
     <xacro:arg name="namespace" default="/" />
     <xacro:property name="description_package" value="$(arg description_package)"/>
     <xacro:property name="show_aruco_board" value="$(arg show_aruco_board)"/>
     <xacro:property name="add_gripper_links" value="$(arg add_gripper_links)"/>
+    <xacro:property name="add_virtual_camera" value="$(arg add_virtual_camera)"/>
     <!-- Import iiwa urdf file -->
     <xacro:include filename="$(find ${description_package})/urdf/iiwa_dual.urdf.xacro" />
@@ -60,5 +61,5 @@
     <link name="base">
         <visual>
-            <origin xyz="-0.5 0 -0.005" rpy="0 0 0" />
+            <origin xyz="-0.6 0 -0.005" rpy="0 0 0" />
             <geometry>
                 <box size="1.5 1 0.01" />
@@ -69,5 +70,5 @@
         </visual>
         <collision>
-            <origin xyz="-0.5 0 -0.005" rpy="0 0 0" />
+            <origin xyz="-0.6 0 -0.005" rpy="0 0 0" />
             <geometry>
                 <box size="1.5 1 0.01" />
@@ -80,4 +81,19 @@
         </inertial>
     </link>
+  <link name="table">
+    <visual>
+      <origin rpy="0.0 0.0 0.0" xyz="0 0 0" />
+      <geometry>
+        <box size="0.75 1.2 0.001" />
+      </geometry>
+      <material name="gray" />
+    </visual>
+    <collision>
+      <origin rpy="0.0 0.0 0.0" xyz="0 0 0" />
+      <geometry>
+        <box size="0.75 1.2 0.001" />
+      </geometry>
+    </collision>
+  </link>
     <joint name="base_to_world" type="fixed">
         <parent link="world"/>
@@ -85,4 +101,10 @@
         <origin xyz="0.0 0.0 0.0" rpy="0.0 0.0 0.0"/>
     </joint>
+     <joint name="world_to_table" type="fixed">
+    <parent link="world" />
+    <child link="table" />
+    <origin rpy="0.0 0.0 0.0" xyz="0.6 0 -0.055" />
+  </joint>
+<xacro:if value="${add_virtual_camera}">
     <link name="camera_pole">
         <visual>
@@ -148,50 +170,51 @@
        <origin xyz="-0.025 0 0" rpy="-1.57 0 1.57" />
     </joint>
-    <xacro:iiwa parent="base" prefix="l_" add_gripper_link="${add_gripper_links}">
+</xacro:if>
+    <xacro:iiwa parent="base" prefix="iiwa_left_" add_gripper_link="${add_gripper_links}">
         <origin xyz="${left_base_frame['x']} ${left_base_frame['y']} ${left_base_frame['z']}"
             rpy="${left_base_frame['roll']} ${left_base_frame['pitch']} ${left_base_frame['yaw']}" />
     </xacro:iiwa>
-    <xacro:iiwa parent="base" prefix="r_" add_gripper_link="${add_gripper_links}">
+    <xacro:iiwa parent="base" prefix="iiwa_right_" add_gripper_link="${add_gripper_links}">
         <origin xyz="${right_base_frame['x']} ${right_base_frame['y']} ${right_base_frame['z']}"
             rpy="${right_base_frame['roll']} ${right_base_frame['pitch']} ${right_base_frame['yaw']}" />
     </xacro:iiwa>
-        <joint name="l_joint_tool1_plate" type="fixed">
+        <joint name="left_joint_tool1_plate" type="fixed">
             <origin rpy="0 0 -1.5708" xyz="0 0 0"/>
-            <parent link="l_tool1"/>
-             <child link="l_plate_link"/>
-             <axis xyz="0 0 0"/>
-         </joint>
-         <link name="l_ee"/>
-          <joint name="l_joint_gripper_ee" type="fixed">
-            <origin xyz="0.027 0 0.168" rpy="0 0.0698 -1.5708"/>
-            <parent link="l_plate_link"/>
-             <child link="l_ee"/>
-             <axis xyz="0 0 0"/>
-         </joint>
-           <joint name="r_joint_tool1_plate" type="fixed">
+            <parent link="iiwa_left_tool1"/>
+             <child link="iiwa_left_plate_link"/>
+             <axis xyz="0 0 0"/>
+         </joint>
+         <link name="iiwa_left_ee"/>
+          <joint name="iiwa_left_joint_gripper_ee" type="fixed">
+            <origin xyz="0.027 0 0.168" rpy="${pi} ${-pi/2 + 0.0698} -1.5708"/>
+            <parent link="iiwa_left_plate_link"/>
+             <child link="iiwa_left_ee"/>
+             <axis xyz="0 0 0"/>
+         </joint>
+           <joint name="iiwa_right_joint_tool1_plate" type="fixed">
             <origin rpy="0 0 1.5708" xyz="0 0 0"/>
-            <parent link="r_tool1"/>
-             <child link="r_plate_link"/>
-             <axis xyz="0 0 0"/>
-         </joint>
-         <link name="r_ee"/>
-          <joint name="r_joint_gripper_ee" type="fixed">
-            <origin xyz="0.027 0 0.168" rpy="0 0.0698 1.5708"/>
-            <parent link="r_plate_link"/>
-             <child link="r_ee"/>
+            <parent link="iiwa_right_tool1"/>
+             <child link="iiwa_right_plate_link"/>
+             <axis xyz="0 0 0"/>
+         </joint>
+         <link name="iiwa_right_ee"/>
+          <joint name="iiwa_right_joint_gripper_ee" type="fixed">
+            <origin xyz="0.027 0 0.168" rpy="${pi} ${-pi/2 + 0.0698} 1.5708"/>
+            <parent link="iiwa_right_plate_link"/>
+             <child link="iiwa_right_ee"/>
              <axis xyz="0 0 0"/>
          </joint>
     <xacro:iiwa_r2c_hardware
-        name="iiwa_left" prefix="l_"
+        name="iiwa_left" prefix="iiwa_left_"
         robot_ip="$(arg robot_ip)" robot_port="$(arg robot_port)"
         command_interface="$(arg command_interface)"
-        initial_positions_file="$(arg initial_positions_file)"
+        initial_positions_file="left_initial_positions.yaml"
         use_sim="$(arg use_sim)" use_fake_hardware="$(arg use_fake_hardware)"
         />
     <xacro:iiwa_r2c_hardware
-        name="iiwa_right" prefix="r_"
+        name="iiwa_right" prefix="iiwa_right_"
         robot_ip="$(arg robot_ip)" robot_port="$(arg robot_port)"
         command_interface="$(arg command_interface)"
-        initial_positions_file="$(arg initial_positions_file)"
+        initial_positions_file="right_initial_positions.yaml"
         use_sim="$(arg use_sim)" use_fake_hardware="$(arg use_fake_hardware)"
         />

File: iiwa_description/ros2_control/iiwa.r2c_hardware.xacro (robot description, xacro)
@@ -24,5 +24,5 @@
                 </hardware>
             </xacro:unless>
-            <joint name="${prefix}joint_a1">
+            <joint name="${prefix}joint_1">
                 <command_interface name="${command_interface}" />
                     <xacro:if value="${command_interface == 'position'}">
@@ -31,5 +31,5 @@
                     </xacro:if>
                 <state_interface name="position">
-                    <param name="initial_value">${initial_positions['joint_a1']}</param>
+                    <param name="initial_value">${initial_positions['joint_1']}</param>
                 </state_interface>
                 <state_interface name="velocity">
@@ -40,5 +40,5 @@
                 </state_interface>
             </joint>
-            <joint name="${prefix}joint_a2">
+            <joint name="${prefix}joint_2">
                 <command_interface name="${command_interface}" />
                     <xacro:if value="${command_interface == 'position'}">
@@ -47,5 +47,5 @@
                     </xacro:if>
                 <state_interface name="position">
-                    <param name="initial_value">${initial_positions['joint_a2']}</param>
+                    <param name="initial_value">${initial_positions['joint_2']}</param>
                 </state_interface>
                 <state_interface name="velocity">
@@ -56,5 +56,5 @@
                 </state_interface>
             </joint>
-            <joint name="${prefix}joint_a3">
+            <joint name="${prefix}joint_3">
                 <command_interface name="${command_interface}" />
                     <xacro:if value="${command_interface == 'position'}">
@@ -63,5 +63,5 @@
                     </xacro:if>
                 <state_interface name="position">
-                    <param name="initial_value">${initial_positions['joint_a3']}</param>
+                    <param name="initial_value">${initial_positions['joint_3']}</param>
                 </state_interface>
                 <state_interface name="velocity">
@@ -72,5 +72,5 @@
                 </state_interface>
             </joint>
-            <joint name="${prefix}joint_a4">
+            <joint name="${prefix}joint_4">
                 <command_interface name="${command_interface}" />
                     <xacro:if value="${command_interface == 'position'}">
@@ -79,5 +79,5 @@
                     </xacro:if>
                 <state_interface name="position">
-                    <param name="initial_value">${initial_positions['joint_a4']}</param>
+                    <param name="initial_value">${initial_positions['joint_4']}</param>
                 </state_interface>
                 <state_interface name="velocity">
@@ -88,5 +88,5 @@
                 </state_interface>
             </joint>
-            <joint name="${prefix}joint_a5">
+            <joint name="${prefix}joint_5">
                 <command_interface name="${command_interface}" />
                     <xacro:if value="${command_interface == 'position'}">
@@ -95,5 +95,5 @@
                     </xacro:if>
                 <state_interface name="position">
-                    <param name="initial_value">${initial_positions['joint_a5']}</param>
+                    <param name="initial_value">${initial_positions['joint_5']}</param>
                 </state_interface>
                 <state_interface name="velocity">
@@ -104,5 +104,5 @@
                 </state_interface>
             </joint>
-            <joint name="${prefix}joint_a6">
+            <joint name="${prefix}joint_6">
                 <command_interface name="${command_interface}" />
                     <xacro:if value="${command_interface == 'position'}">
@@ -111,5 +111,5 @@
                     </xacro:if>
                 <state_interface name="position">
-                    <param name="initial_value">${initial_positions['joint_a6']}</param>
+                    <param name="initial_value">${initial_positions['joint_6']}</param>
                 </state_interface>
                 <state_interface name="velocity">
@@ -120,5 +120,5 @@
                 </state_interface>
             </joint>
-            <joint name="${prefix}joint_a7">
+            <joint name="${prefix}joint_7">
                 <command_interface name="${command_interface}" />
                     <xacro:if value="${command_interface == 'position'}">
@@ -127,5 +127,5 @@
                     </xacro:if>
                 <state_interface name="position">
-                    <param name="initial_value">${initial_positions['joint_a7']}</param>
+                    <param name="initial_value">${initial_positions['joint_7']}</param>
                 </state_interface>
                 <state_interface name="velocity">
@@ -137,11 +137,11 @@
             </joint>
             <sensor name="${prefix}external_torque_sensor">
-                <state_interface name="external_torque.joint_a1"/>
-                <state_interface name="external_torque.joint_a2"/>
-                <state_interface name="external_torque.joint_a3"/>
-                <state_interface name="external_torque.joint_a4"/>
-                <state_interface name="external_torque.joint_a5"/>
-                <state_interface name="external_torque.joint_a6"/>
-                <state_interface name="external_torque.joint_a7"/>
+                <state_interface name="external_torque.joint_1"/>
+                <state_interface name="external_torque.joint_2"/>
+                <state_interface name="external_torque.joint_3"/>
+                <state_interface name="external_torque.joint_4"/>
+                <state_interface name="external_torque.joint_5"/>
+                <state_interface name="external_torque.joint_6"/>
+                <state_interface name="external_torque.joint_7"/>
             </sensor>
         </ros2_control>

File: iiwa_description/srdf/iiwa_dual.srdf.xacro (robot description, xacro)
@@ -13,19 +13,19 @@
   <disable_collisions link1="marker_link_0" link2="r_link_7" reason="Adjacent" />
   <disable_collisions link1="marker_link_0" link2="r_link_6" reason="Adjacent" />
-  <group_state name="calibration" group="r_iiwa_arm">
-        <joint name="r_joint_a1" value="-0.08010961654547082"/>
-        <joint name="r_joint_a2" value="-0.16420504552657098"/>
-        <joint name="r_joint_a3" value="-0.27250731500631165"/>
-        <joint name="r_joint_a4" value="1.8724710663682194"/>
-        <joint name="r_joint_a5" value="1.2174080270970293"/>
-        <joint name="r_joint_a6" value="1.2045682076607263"/>
-        <joint name="r_joint_a7" value="-0.11062877843161172"/>
+  <group_state name="calibration" group="iiwa_right_arm">
+        <joint name="iiwa_right_joint_1" value="-0.08010961654547082"/>
+        <joint name="iiwa_right_joint_2" value="-0.16420504552657098"/>
+        <joint name="iiwa_right_joint_3" value="-0.27250731500631165"/>
+        <joint name="iiwa_right_joint_4" value="1.8724710663682194"/>
+        <joint name="iiwa_right_joint_5" value="1.2174080270970293"/>
+        <joint name="iiwa_right_joint_6" value="1.2045682076607263"/>
+        <joint name="iiwa_right_joint_7" value="-0.11062877843161172"/>
  </group_state>
   </xacro:if>
-  <xacro:iiwa_srdf name="$(arg name)" prefix="l_" base="base"/>
-  <xacro:iiwa_srdf name="$(arg name)" prefix="r_" base="base"/>
+  <xacro:iiwa_srdf name="arm" prefix="iiwa_left_" base="base"/>
+  <xacro:iiwa_srdf name="arm" prefix="iiwa_right_" base="base"/>
   <group name="dual_arm">
-    <group name="l_iiwa_arm" />
-    <group name="r_iiwa_arm" />
+    <group name="iiwa_left_arm" />
+    <group name="iiwa_right_arm" />
   </group>
 </robot>

File: iiwa_description/srdf/iiwa_dual_macro.srdf.xacro (robot description, xacro)
@@ -2,35 +2,32 @@
 <robot xmlns:xacro="http://www.ros.org/wiki/xacro">
   <xacro:macro name="iiwa_srdf" params="name prefix base">
-     <group name="${prefix}${name}_arm">
-        <chain base_link="${prefix}iiwa_base" tip_link="${prefix}tool0" />
+     <group name="${prefix}${name}">
+        <chain base_link="${prefix}base" tip_link="${prefix}tool0" />
     </group>
-     <group name="${prefix}${name}_arm_ee">
-        <chain base_link="${prefix}iiwa_base" tip_link="${prefix}ee" />
+     <group name="${prefix}${name}_ee">
+        <chain base_link="${prefix}base" tip_link="${prefix}ee" />
     </group>
-    <group_state name="ready" group="${prefix}${name}_arm">
-        <joint name="${prefix}joint_a1" value="0"/>
-        <joint name="${prefix}joint_a2" value="-0.785"/>
-        <joint name="${prefix}joint_a3" value="0"/>
-        <joint name="${prefix}joint_a4" value="-2.356"/>
-        <joint name="${prefix}joint_a5" value="0"/>
-        <joint name="${prefix}joint_a6" value="1.571"/>
-        <joint name="${prefix}joint_a7" value="0.785"/>
+    <group_state name="ready" group="${prefix}${name}">
+        <joint name="${prefix}joint_1" value="0"/>
+        <joint name="${prefix}joint_2" value="-0.785"/>
+        <joint name="${prefix}joint_3" value="0"/>
+        <joint name="${prefix}joint_4" value="-2.356"/>
+        <joint name="${prefix}joint_5" value="0"/>
+        <joint name="${prefix}joint_6" value="1.571"/>
+        <joint name="${prefix}joint_7" value="0.785"/>
     </group_state>
-     <group_state name="upright" group="${prefix}${name}_arm">
-        <joint name="${prefix}joint_a1" value="0"/>
-        <joint name="${prefix}joint_a2" value="0"/>
-        <joint name="${prefix}joint_a3" value="0"/>
-        <joint name="${prefix}joint_a4" value="0"/>
-        <joint name="${prefix}joint_a5" value="0"/>
-        <joint name="${prefix}joint_a6" value="0"/>
-        <joint name="${prefix}joint_a7" value="0"/>
+     <group_state name="upright" group="${prefix}${name}">
+        <joint name="${prefix}joint_1" value="0"/>
+        <joint name="${prefix}joint_2" value="0"/>
+        <joint name="${prefix}joint_3" value="0"/>
+        <joint name="${prefix}joint_4" value="0"/>
+        <joint name="${prefix}joint_5" value="0"/>
+        <joint name="${prefix}joint_6" value="0"/>
+        <joint name="${prefix}joint_7" value="0"/>
     </group_state>
-    <disable_collisions link1="${base}" link2="${prefix}link_0" reason="Adjacent" />
-    <disable_collisions link1="${base}" link2="${prefix}link_1" reason="Never" />
-    <disable_collisions link1="${base}" link2="${prefix}link_2" reason="Never" />
-    <disable_collisions link1="${prefix}iiwa_base" link2="${prefix}link_0" reason="Adjacent" />
-    <disable_collisions link1="${prefix}iiwa_base" link2="${prefix}link_1" reason="Never" />
-    <disable_collisions link1="${prefix}iiwa_base" link2="${prefix}link_2" reason="Never" />
-    <disable_collisions link1="${prefix}iiwa_base" link2="${prefix}link_3" reason="Never" />
+    <disable_collisions link1="${prefix}base" link2="${prefix}link_0" reason="Adjacent" />
+    <disable_collisions link1="${prefix}base" link2="${prefix}link_1" reason="Never" />
+    <disable_collisions link1="${prefix}base" link2="${prefix}link_2" reason="Never" />
+    <disable_collisions link1="${prefix}base" link2="${prefix}link_3" reason="Never" />
     <disable_collisions link1="${prefix}link_0" link2="${prefix}link_1" reason="Adjacent" />
     <disable_collisions link1="${prefix}link_0" link2="${prefix}link_2" reason="Never" />

File: iiwa_description/urdf/iiwa_dual.urdf.xacro (robot description, xacro)
@@ -5,13 +5,13 @@
 <xacro:property name="gripper_width" value="0.1" />
 <xacro:property name="gripper_depth" value="0.01" />
-  <link name="${prefix}iiwa_base" type="fixed"/>
-  <joint name="${prefix}iiwa_root_joint" type="fixed">
+  <link name="${prefix}base" type="fixed"/>
+  <joint name="${prefix}_root_joint" type="fixed">
       <xacro:insert_block name="origin" />
       <parent link="${parent}"/>
-      <child link="${prefix}iiwa_base"/>
-  </joint>
-  <joint name="${prefix}iiwa_base_joint" type="fixed">
+      <child link="${prefix}base"/>
+  </joint>
+  <joint name="${prefix}base_joint" type="fixed">
       <origin rpy="0.0 0 0" xyz="0 0 0"/>
-      <parent link="${prefix}iiwa_base"/>
+      <parent link="${prefix}base"/>
       <child link="${prefix}link_0"/>
   </joint>
@@ -223,5 +223,5 @@
   <link name="${prefix}tool0"/>
   <link name="${prefix}tool1"/>
-  <joint name="${prefix}joint_a1" type="revolute">
+  <joint name="${prefix}joint_1" type="revolute">
       <origin rpy="0 0 0" xyz="0 0 0"/>
       <parent link="${prefix}link_0"/>
@@ -230,5 +230,5 @@
       <limit effort="320" lower="-2.9668" upper="2.9668" velocity="1.4834"/>
   </joint>
-  <joint name="${prefix}joint_a2" type="revolute">
+  <joint name="${prefix}joint_2" type="revolute">
       <origin rpy="0 0 0" xyz="-0.00043624 0 0.36"/>
       <parent link="${prefix}link_1"/>
@@ -237,5 +237,5 @@
       <limit effort="320" lower="-2.0942" upper="2.0942" velocity="1.4834"/>
   </joint>
-  <joint name="${prefix}joint_a3" type="revolute">
+  <joint name="${prefix}joint_3" type="revolute">
       <origin rpy="0 0 0" xyz="0 0 0"/>
       <parent link="${prefix}link_2"/>
@@ -244,5 +244,5 @@
       <limit effort="176" lower="-2.9668" upper="2.9668" velocity="1.7452"/>
   </joint>
-  <joint name="${prefix}joint_a4" type="revolute">
+  <joint name="${prefix}joint_4" type="revolute">
       <origin rpy="0 0 0" xyz="0.00043624 0 0.42"/>
       <parent link="${prefix}link_3"/>
@@ -251,5 +251,5 @@
       <limit effort="176" lower="-2.0942" upper="2.0942" velocity="1.3089"/>
   </joint>
-  <joint name="${prefix}joint_a5" type="revolute">
+  <joint name="${prefix}joint_5" type="revolute">
       <origin rpy="0 0 0" xyz="0 0 0"/>
       <parent link="${prefix}link_4"/>
@@ -258,5 +258,5 @@
       <limit effort="110" lower="-2.9668" upper="2.9668" velocity="2.2688"/>
   </joint>
-  <joint name="${prefix}joint_a6" type="revolute">
+  <joint name="${prefix}joint_6" type="revolute">
       <origin rpy="0 0 0" xyz="0 0 0.4"/>
       <parent link="${prefix}link_5"/>
@@ -265,5 +265,5 @@
       <limit effort="40" lower="-2.0942" upper="2.0942" velocity="2.356"/>
   </joint>
-  <joint name="${prefix}joint_a7" type="revolute">
+  <joint name="${prefix}joint_7" type="revolute">
       <origin rpy="0 0 0" xyz="0 0 0"/>
       <parent link="${prefix}link_6"/>
@@ -272,5 +272,5 @@
       <limit effort="40" lower="-3.0541" upper="3.0541" velocity="2.356"/>
   </joint>
-  <joint name="${prefix}joint_a7-tool0" type="fixed">
+  <joint name="${prefix}joint_7-tool0" type="fixed">
       <origin rpy="0 0 0" xyz="0 0 0.152"/>
       <parent link="${prefix}link_7"/>

Commit message: gripper frame

File: iiwa_description/config/iiwa_dual.config.xacro (robot description, xacro)
@@ -187,5 +187,5 @@
          <link name="iiwa_left_ee"/>
           <joint name="iiwa_left_joint_gripper_ee" type="fixed">
-            <origin xyz="0.027 0 0.168" rpy="${pi} ${-pi/2 + 0.0698} -1.5708"/>
+            <origin xyz="0.027 0 0.168" rpy="${0} ${-pi/2 + 0.0698} -1.5708"/>
             <parent link="iiwa_left_plate_link"/>
              <child link="iiwa_left_ee"/>
@@ -200,5 +200,5 @@
          <link name="iiwa_right_ee"/>
           <joint name="iiwa_right_joint_gripper_ee" type="fixed">
-            <origin xyz="0.027 0 0.168" rpy="${pi} ${-pi/2 + 0.0698} 1.5708"/>
+            <origin xyz="0.027 0 0.168" rpy="${0} ${-pi/2 + 0.0698} 1.5708"/>
             <parent link="iiwa_right_plate_link"/>
              <child link="iiwa_right_ee"/>
