Commit message: tactile skin

File: iiwa_description/config/iiwa_dual.config.xacro (robot description, xacro)
@@ -104,6 +104,75 @@
     <parent link="world" />
     <child link="table" />
-    <origin rpy="0.0 0.0 0.0" xyz="0.6 0 -0.055" />
-  </joint>
+    <origin rpy="0.008 0.004 3.139" xyz="0.869 -0.053 -0.050" />
+    <!--<origin rpy="0.0 0.0 0.0" xyz="0.6 0 -0.055" />-->
+  </joint>
+  <joint name="iiwa_left_link_6_to_tactile_skin_bracket" type="fixed">
+    <parent link="iiwa_left_link_6" />
+    <child link="iiwa_left_tactile_skin_bracket" />
+    <origin rpy="-0 0 0.0" xyz="0 0 0" />
+  </joint>
+  <link name="iiwa_left_tactile_skin_bracket">
+    <visual>
+        <origin rpy="0 0 0" xyz="0.1302 -0.0167 -0.64179"/>
+      <geometry>
+        <mesh filename="package://iiwa_description/meshes/tactile_skin/tactile_skin_bracket.stl" scale="0.001 0.001 0.001"/>
+      </geometry>
+    </visual>
+     <collision>
+        <origin rpy="0 0 0" xyz="0.1302 -0.0167 -0.64179"/>
+      <geometry>
+        <mesh filename="package://iiwa_description/meshes/tactile_skin/tactile_skin_bracket.stl" scale="0.001 0.001 0.001"/>
+      </geometry>
+    </collision>
+  </link>
+  <joint name="iiwa_left_tactile_skin_joint" type="fixed">
+    <parent link="iiwa_left_tactile_skin_bracket" />
+    <child link="iiwa_left_tactile_skin" />
+    <origin rpy="0 1.5707963267948966 0" xyz="0 0.015 0.0445" />
+  </joint>
+     <joint name="iiwa_left_tactile_skin_center_joint" type="fixed">
+    <parent link="iiwa_left_tactile_skin_bracket"/>
+    <child link="iiwa_left_tactile_skin_center"/>
+    <origin rpy="0 0 0" xyz="0 0.07 0"/>
+  </joint>
+  <link name="iiwa_left_tactile_skin_center"/>
+  <link name="iiwa_left_tactile_skin"/>
+  <joint name="iiwa_right_link_6_to_tactile_skin_bracket" type="fixed">
+    <parent link="iiwa_right_link_6" />
+    <child link="iiwa_right_tactile_skin_bracket" />
+    <origin rpy="0.0 0.0 0.0" xyz="0 0 0" />
+  </joint>
+  <link name="iiwa_right_tactile_skin_bracket">
+    <visual>
+        <origin rpy="0 0 0" xyz=" 0.1302 -0.0167 -0.6417900000000001"/>
+      <geometry>
+        <mesh filename="package://iiwa_description/meshes/tactile_skin/tactile_skin_bracket.stl" scale="0.001 0.001 0.001"/>
+      </geometry>
+    </visual>
+    <collision>
+        <origin rpy="0 0 0" xyz=" 0.1302 -0.0167 -0.6417900000000001"/>
+      <geometry>
+        <mesh filename="package://iiwa_description/meshes/tactile_skin/tactile_skin_bracket.stl" scale="0.001 0.001 0.001"/>
+      </geometry>
+    </collision>
+  </link>
+  <joint name="iiwa_right_tactile_skin_joint" type="fixed">
+    <parent link="iiwa_right_tactile_skin_bracket" />
+    <child link="iiwa_right_tactile_skin" />
+    <origin rpy="3.141592653589793 -1.5707963267948966 0" xyz="0 0.009999999999999998 -0.04450000000000001" />
+  </joint>
+  <joint name="iiwa_right_tactile_skin_center_joint" type="fixed">
+    <parent link="iiwa_right_tactile_skin_bracket"/>
+    <child link="iiwa_right_tactile_skin_center"/>
+    <origin rpy="0 0 0" xyz="0 0.07 0"/>
+  </joint>
+  <link name="iiwa_right_tactile_skin_center"/>
+  <link name="iiwa_right_tactile_skin"/>
+  <joint name="world_to_camera_213322070245_color_optical_frame" type="fixed">
+    <parent link="world"/>
+    <child link="camera_213322070245_color_optical_frame"/>
+    <origin rpy="-2.436 -0.007 -1.575" xyz="-0.221 0.026 1.026"/>
+  </joint>
+  <link name="camera_213322070245_color_optical_frame"/>
 <xacro:if value="${add_virtual_camera}">
     <link name="camera_pole">

File: iiwa_description/srdf/iiwa_dual_macro.srdf.xacro (robot description, xacro)
@@ -58,4 +58,5 @@
     <disable_collisions link1="${prefix}ft_sensor_link" link2="${prefix}link_7" reason="Adjacent" />
     <disable_collisions link1="${prefix}ft_sensor_link" link2="${prefix}plate_link" reason="Adjacent" />
+    <disable_collisions link1="${prefix}link_6" link2="${prefix}tactile_skin_bracket" reason="Adjacent" />
   </xacro:macro>
 </robot>

Commit message: tactile skin end effectors

File: iiwa_description/config/iiwa_dual.config.xacro (robot description, xacro)
@@ -133,8 +133,8 @@
      <joint name="iiwa_left_tactile_skin_center_joint" type="fixed">
     <parent link="iiwa_left_tactile_skin_bracket"/>
-    <child link="iiwa_left_tactile_skin_center"/>
-    <origin rpy="0 0 0" xyz="0 0.07 0"/>
-  </joint>
-  <link name="iiwa_left_tactile_skin_center"/>
+    <child link="iiwa_left_tactile_ee"/>
+    <origin rpy="0 -${pi/2} 0" xyz="0 0.07 0"/>
+  </joint>
+  <link name="iiwa_left_tactile_ee"/>
   <link name="iiwa_left_tactile_skin"/>
   <joint name="iiwa_right_link_6_to_tactile_skin_bracket" type="fixed">
@@ -164,10 +164,9 @@
   <joint name="iiwa_right_tactile_skin_center_joint" type="fixed">
     <parent link="iiwa_right_tactile_skin_bracket"/>
-    <child link="iiwa_right_tactile_skin_center"/>
-    <origin rpy="0 0 0" xyz="0 0.07 0"/>
-  </joint>
-  <link name="iiwa_right_tactile_skin_center"/>
+    <child link="iiwa_right_tactile_ee"/>
+   <origin rpy="${pi} -${pi/2} 0" xyz="0 0.07 0"/>
+  </joint>
+  <link name="iiwa_right_tactile_ee"/>
   <link name="iiwa_right_tactile_skin"/>
- <!--
   <joint name="world_to_camera_213322070245_color_optical_frame" type="fixed">
     <parent link="world"/>
@@ -176,5 +175,4 @@
   </joint>
   <link name="camera_213322070245_color_optical_frame"/>
--->
 <xacro:if value="${add_virtual_camera}">
     <link name="camera_pole">

File: iiwa_description/srdf/iiwa_dual_macro.srdf.xacro (robot description, xacro)
@@ -7,4 +7,7 @@
      <group name="${prefix}${name}_ee">
         <chain base_link="${prefix}base" tip_link="${prefix}ee" />
+    </group>
+     <group name="${prefix}${name}_tactile">
+        <chain base_link="${prefix}base" tip_link="${prefix}tactile_ee" />
     </group>
     <group_state name="ready" group="${prefix}${name}">

Commit message: update-plate-grippers-and-camera

File: iiwa_description/config/iiwa_dual.config.xacro (robot description, xacro)
@@ -172,5 +172,5 @@
     <parent link="world"/>
     <child link="camera_213322070245_color_optical_frame"/>
-    <origin rpy="-2.436 -0.007 -1.575" xyz="-0.221 0.026 1.026"/>
+    <origin rpy="-2.424 0.013 -1.605" xyz="-0.261 0.010 1.031"/>
   </joint>
   <link name="camera_213322070245_color_optical_frame"/>
@@ -249,5 +249,5 @@
     </xacro:iiwa>
         <joint name="left_joint_tool1_plate" type="fixed">
-            <origin rpy="0 0 -1.5708" xyz="0 0 0"/>
+            <origin rpy="0 0 -0.785398" xyz="0 0 0"/>
             <parent link="iiwa_left_tool1"/>
              <child link="iiwa_left_plate_link"/>
@@ -262,5 +262,5 @@
          </joint>
            <joint name="iiwa_right_joint_tool1_plate" type="fixed">
-            <origin rpy="0 0 1.5708" xyz="0 0 0"/>
+            <origin rpy="0 0 -0.785398" xyz="0 0 0"/>
             <parent link="iiwa_right_tool1"/>
              <child link="iiwa_right_plate_link"/>
